Commit message: 修复了rviz中反向移动的问题

File: src/wheeltec_robot_urdf/urdf/mini_mec_robot.urdf (robot description, URDF)
Before this commit: robot mini_mec_robot, 8 links, 7 joints
Joints:
- joint laser_joint: origin xyz=0.0316310367407428 9.05810809802502E-05 0.095024183741431 rpy=0 0 3.14159265358979 -> xyz=0.0316310367407428 9.05810809802502E-05 0.095024183741431 rpy=0 0 0
